Commit message: Update race car, camera, and track

File: line_follower/urdf/mogi_bot.xacro (robot description, xacro)
@@ -1,28 +1,28 @@
 <?xml version='1.0'?>
 <robot name="mogi_bot" xmlns:xacro="http://www.ros.org/wiki/xacro">
-  <!-- Gazebo plugin -->
-  <xacro:include filename="$(find line_follower_race_car)/urdf/mogi_bot.gazebo" />
-  <!-- RViz colors -->
-  <xacro:include filename="$(find line_follower_race_car)/urdf/materials.xacro" />
+  <!-- STEP 3 - Gazebo plugin -->
+  <xacro:include filename="$(find line_follower)/urdf/mogi_bot.gazebo" />
+  <!-- STEP 4 - RViz colors -->
+  <xacro:include filename="$(find line_follower)/urdf/materials.xacro" />
+  <!-- STEP 1 - Robot chassis -->
   <link name="base_footprint"></link>
   <joint name="base_footprint_joint" type="fixed">
-    <origin xyz="0 0 0" rpy="0 0 0" />
+    <origin xyz="0 0 0" rpy="0 0 -1.5707" />
     <parent link="base_footprint"/>
     <child link="base_link" />
   </joint>
-  <!-- Robot chassis -->
   <link name='base_link'>
     <pose>0 0 0.1 0 0 0</pose>
     <inertial>
       <mass value="15.0"/>
-      <origin xyz="0.0 0 0" rpy="0 0 0"/>
-      <inertia
-          ixx="0.1" ixy="0" ixz="0"
-          iyy="0.1" iyz="0"
-          izz="0.1"
-      />
-    </inertial>
-    <collision name='collision'>
-      <origin xyz="0 0 0" rpy="0 0 0"/>
+      <origin xyz="0.0 0 0" rpy=" 0 0 0"/>
+      <inertia
+          ixx="0.1" ixy="0" ixz="0"
+          iyy="0.1" iyz="0"
+          izz="0.1"
+      />
+    </inertial>
+    <collision name='collision'>
+      <origin xyz="0 0 0" rpy=" 0 0 -1.5707"/>
       <geometry>
         <box size=".4 .2 .1"/>
@@ -30,106 +30,147 @@
     </collision>
     <visual name='base_link_visual'>
-      <origin xyz="0 0 0" rpy="0 0 0"/>
+      <origin xyz="0 0 0" rpy=" 0 0 -1.5707"/>
       <geometry>
         <!--box size=".4 .2 .1"/-->
-        <mesh filename = "package://line_follower_race_car/meshes/mogi_bot.dae"/>
-      </geometry>
-      <material name="orange"/>
-    </visual>
-    <collision name='rear_caster_collision'>
-      <origin xyz="-0.15 0 -0.05" rpy="0 0 0"/>
-      <geometry>
-        <sphere radius="0.0499"/>
-      </geometry>
-    </collision>
-    <visual name='rear_caster_visual'>
-      <origin xyz="-0.15 0 -0.05" rpy="0 0 0"/>
-      <geometry>
-        <sphere radius="0.05"/>
-      </geometry>
-    </visual>
-    <collision name='front_caster_collision'>
-      <origin xyz="0.15 0 -0.05" rpy="0 0 0"/>
-      <geometry>
-        <sphere radius="0.0499"/>
-      </geometry>
-    </collision>
-    <visual name='front_caster_visual'>
-      <origin xyz="0.15 0 -0.05" rpy="0 0 0"/>
-      <geometry>
-        <sphere radius="0.05"/>
-      </geometry>
-    </visual>
-  </link>
-  <!-- Wheels -->
-  <joint type="continuous" name="left_wheel_joint">
-    <origin xyz="0 0.15 0" rpy="0 0 0"/>
-    <child link="left_wheel"/>
-    <parent link="base_link"/>
-    <axis xyz="0 1 0" rpy="0 0 0"/>
-    <limit effort="10000" velocity="1000"/>
-    <dynamics damping="1.0" friction="1.0"/>
-  </joint>
-  <link name='left_wheel'>
-    <inertial>
-      <mass value="5.0"/>
-      <origin xyz="0 0 0" rpy="0 1.5707 1.5707"/>
-      <inertia
-          ixx="0.1" ixy="0" ixz="0"
-          iyy="0.1" iyz="0"
-          izz="0.1"
-      />
-    </inertial>
-    <collision name='collision'>
-      <origin xyz="0 0 0" rpy="0 1.5707 1.5707"/>
-      <geometry>
-        <cylinder radius=".1" length=".05"/>
-      </geometry>
-    </collision>
-    <visual name='left_wheel_visual'>
-      <origin xyz="0 0 0" rpy="0 1.5707 1.5707"/>
-      <geometry>
-        <!--cylinder radius=".1" length=".05"/-->
-        <mesh filename = "package://line_follower_race_car/meshes/wheel.dae"/>
-      </geometry>
-      <material name="green"/>
-    </visual>
-  </link>
-  <joint type="continuous" name="right_wheel_joint">
-    <origin xyz="0 -0.15 0" rpy="0 0 0"/>
-    <child link="right_wheel"/>
-    <parent link="base_link"/>
-    <axis xyz="0 1 0" rpy="0 0 0"/>
-    <limit effort="10000" velocity="1000"/>
-    <dynamics damping="1.0" friction="1.0"/>
-  </joint>
-  <link name='right_wheel'>
-    <inertial>
-      <mass value="5.0"/>
-      <origin xyz="0 0 0" rpy="0 1.5707 1.5707"/>
-      <inertia
-          ixx="0.1" ixy="0" ixz="0"
-          iyy="0.1" iyz="0"
-          izz="0.1"
-      />
-    </inertial>
-    <collision name='collision'>
-      <origin xyz="0 0 0" rpy="0 1.5707 1.5707"/>
-      <geometry>
-        <cylinder radius=".1" length=".05"/>
-      </geometry>
-    </collision>
-    <visual name='right_wheel_visual'>
-      <origin xyz="0 0 0" rpy="0 1.5707 1.5707"/>
-      <geometry>
-        <!--cylinder radius=".1" length=".05"/-->
-        <mesh filename = "package://line_follower_race_car/meshes/wheel.dae"/>
-      </geometry>
-      <material name="green"/>
+        <mesh filename = "package://line_follower/meshes/body.dae"/>
+      </geometry>
+    </visual>
+  </link>
+  <!-- STEP 2 - Wheels -->
+  <!-- Front left -->
+  <joint type="continuous" name="front_left_wheel_joint">
+    <origin xyz="0.23 0.17 0" rpy="0 0 0"/>
+    <child link="front_left_wheel"/>
+    <parent link="base_link"/>
+    <axis xyz="0 1 0" rpy="0 0 0"/>
+    <limit effort="10000" velocity="1000"/>
+    <dynamics damping="1.0" friction="1.0"/>
+  </joint>
+  <link name='front_left_wheel'>
+    <inertial>
+      <mass value="5.0"/>
+      <origin xyz="0 0 0" rpy="0 1.5707 1.5707"/>
+      <inertia
+          ixx="0.1" ixy="0" ixz="0"
+          iyy="0.1" iyz="0"
+          izz="0.1"
+      />
+    </inertial>
+    <collision name='collision'>
+      <origin xyz="0 0 0" rpy="0 1.5707 1.5707"/>
+      <geometry>
+        <cylinder radius=".1" length=".05"/>
+      </geometry>
+    </collision>
+    <visual name='front_left_wheel_visual'>
+      <origin xyz="0 0 0" rpy="0 1.5707 1.5707"/>
+      <geometry>
+        <!--cylinder radius=".1" length=".05"/-->
+        <mesh filename = "package://line_follower/meshes/front_wheels.dae"/>
+      </geometry>
+    </visual>
+  </link>
+<!-- Front right -->
+  <joint type="continuous" name="front_right_wheel_joint">
+    <origin xyz="0.23 -0.19 0" rpy="0 0 0"/>
+    <child link="front_right_wheel"/>
+    <parent link="base_link"/>
+    <axis xyz="0 1 0" rpy="0 0 0"/>
+    <limit effort="10000" velocity="1000"/>
+    <dynamics damping="1.0" friction="1.0"/>
+  </joint>
+  <link name='front_right_wheel'>
+    <inertial>
+      <mass value="5.0"/>
+      <origin xyz="0 0 0" rpy="0 1.5707 -1.5707"/>
+      <inertia
+          ixx="0.1" ixy="0" ixz="0"
+          iyy="0.1" iyz="0"
+          izz="0.1"
+      />
+    </inertial>
+    <collision name='collision'>
+      <origin xyz="0 0 0" rpy="0 1.5707 -1.5707"/>
+      <geometry>
+        <cylinder radius=".1" length=".05"/>
+      </geometry>
+    </collision>
+    <visual name='front_right_wheel_visual'>
+      <origin xyz="0 0 0" rpy="0 1.5707 -1.5707"/>
+      <geometry>
+        <!--cylinder radius=".1" length=".05"/-->
+        <mesh filename = "package://line_follower/meshes/front_wheels.dae"/>
+      </geometry>
+    </visual>
+  </link>
+<!-- Rear left -->
+  <joint type="continuous" name="rear_left_wheel_joint">
+    <origin xyz="-0.25 0.17 0" rpy="0 0 0"/>
+    <child link="rear_left_wheel"/>
+    <parent link="base_link"/>
+    <axis xyz="0 1 0" rpy="0 0 0"/>
+    <limit effort="10000" velocity="1000"/>
+    <dynamics damping="1.0" friction="1.0"/>
+  </joint>
+  <link name='rear_left_wheel'>
+    <inertial>
+      <mass value="5.0"/>
+      <origin xyz="0 0 0" rpy="0 1.5707 1.5707"/>
+      <inertia
+          ixx="0.1" ixy="0" ixz="0"
+          iyy="0.1" iyz="0"
+          izz="0.1"
+      />
+    </inertial>
+    <collision name='collision'>
+      <origin xyz="0 0 0" rpy="0 1.5707 1.5707"/>
+      <geometry>
+        <cylinder radius=".1" length=".05"/>
+      </geometry>
+    </collision>
+    <visual name='rear_left_wheel_visual'>
+      <origin xyz="0 0 0" rpy="0 1.5707 1.5707"/>
+      <geometry>
+        <!--cylinder radius=".1" length=".05"/-->
+        <mesh filename = "package://line_follower/meshes/front_wheels.dae"/>
+      </geometry>
+    </visual>
+  </link>
+<!-- Rear right -->
+  <joint type="continuous" name="rear_right_wheel_joint">
+    <origin xyz="-0.25 -0.19 0" rpy="0 0 0"/>
+    <child link="rear_right_wheel"/>
+    <parent link="base_link"/>
+    <axis xyz="0 1 0" rpy="0 0 0"/>
+    <limit effort="10000" velocity="1000"/>
+    <dynamics damping="1.0" friction="1.0"/>
+  </joint>
+  <link name='rear_right_wheel'>
+    <inertial>
+      <mass value="5.0"/>
+      <origin xyz="0 0 0" rpy="0 1.5707 -1.5707"/>
+      <inertia
+          ixx="0.1" ixy="0" ixz="0"
+          iyy="0.1" iyz="0"
+          izz="0.1"
+      />
+    </inertial>
+    <collision name='collision'>
+      <origin xyz="0 0 0" rpy="0 1.5707 -1.5707"/>
+      <geometry>
+        <cylinder radius=".1" length=".05"/>
+      </geometry>
+    </collision>
+    <visual name='rear_right_wheel_visual'>
+      <origin xyz="0 0 0" rpy="0 1.5707 -1.5707"/>
+      <geometry>
+        <!--cylinder radius=".1" length=".05"/-->
+        <mesh filename = "package://line_follower/meshes/front_wheels.dae"/>
+      </geometry>
     </visual>
   </link>
     <!-- Camera -->
   <joint type="fixed" name="camera_joint">
-    <origin xyz="0.225 0 0.075" rpy="0 0 0"/>
+    <origin xyz="0.350 -0.005 0.075" rpy="0 0 0"/>
     <child link="camera_link"/>
     <parent link="base_link"/>
@@ -170,41 +211,3 @@
   <link name="camera_link_optical">
   </link>
-  <!-- IMU -->
-  <joint name="imu_joint" type="fixed">
-    <origin xyz="0 0 0" rpy="0 0 0" />
-    <parent link="base_link"/>
-    <child link="imu_link" />
-  </joint>
-  <link name="imu_link">
-  </link>
-  <!-- Lidar -->
-  <joint type="fixed" name="scan_joint">
-    <origin xyz="0.0 0 0.15" rpy="0 0 0"/>
-    <child link="scan_link"/>
-    <parent link="base_link"/>
-    <axis xyz="0 1 0" rpy="0 0 0"/>
-  </joint>
-  <link name='scan_link'>
-    <inertial>
-      <mass value="1e-5"/>
-      <origin xyz="0 0 0" rpy="0 0 0"/>
-      <inertia
-          ixx="1e-6" ixy="0" ixz="0"
-          iyy="1e-6" iyz="0"
-          izz="1e-6"
-      />
-    </inertial>
-    <collision name='collision'>
-      <origin xyz="0 0 0" rpy="0 0 0"/>
-      <geometry>
-        <box size=".1 .1 .1"/>
-      </geometry>
-    </collision>
-    <visual name='scan_link_visual'>
-      <origin xyz="0 0 0" rpy="0 0 0"/>
-      <geometry>
-        <mesh filename = "package://line_follower_race_car/meshes/lidar.dae"/>
-      </geometry>
-    </visual>
-  </link>
 </robot>

Commit message: Skid steer control

File: line_follower/urdf/mogi_bot.xacro (robot description, xacro)
@@ -8,5 +8,5 @@
   <link name="base_footprint"></link>
   <joint name="base_footprint_joint" type="fixed">
-    <origin xyz="0 0 0" rpy="0 0 -1.5707" />
+    <origin xyz="0 0 0" rpy="0 0 0" />
     <parent link="base_footprint"/>
     <child link="base_link" />
@@ -211,3 +211,44 @@
   <link name="camera_link_optical">
   </link>
+  <!-- STEP 7 - Gazebo physics -->
+  <gazebo reference="front_left_wheel">
+    <!-- kp and kd for rubber -->
+    <kp>1000000.0</kp>
+    <kd>100.0</kd>
+    <mu1>1.5</mu1>
+    <mu2>1.5</mu2>
+    <fdir1>1 0 0</fdir1>
+    <maxVel>1.0</maxVel>
+    <minDepth>0.00</minDepth>
+  </gazebo>
+  <gazebo reference="front_right_wheel">
+    <!-- kp and kd for rubber -->
+    <kp>1000000.0</kp>
+    <kd>100.0</kd>
+    <mu1>1.5</mu1>
+    <mu2>1.5</mu2>
+    <fdir1>1 0 0</fdir1>
+    <maxVel>1.0</maxVel>
+    <minDepth>0.00</minDepth>
+  </gazebo>
+  <gazebo reference="rear_left_wheel">
+    <!-- kp and kd for rubber -->
+    <kp>1000000.0</kp>
+    <kd>100.0</kd>
+    <mu1>1.5</mu1>
+    <mu2>1.5</mu2>
+    <fdir1>1 0 0</fdir1>
+    <maxVel>1.0</maxVel>
+    <minDepth>0.00</minDepth>
+  </gazebo>
+  <gazebo reference="rear_right_wheel">
+    <!-- kp and kd for rubber -->
+    <kp>1000000.0</kp>
+    <kd>100.0</kd>
+    <mu1>1.5</mu1>
+    <mu2>1.5</mu2>
+    <fdir1>1 0 0</fdir1>
+    <maxVel>1.0</maxVel>
+    <minDepth>0.00</minDepth>
+  </gazebo>
 </robot>
